File: M17_GM300_RPi.sch (KiCad schematic (older format))
At the start: 44 parts, among them J1 RJ45, J2 Conn_01x06_Male, J3 RPi_SND, J4 Conn_01x20_Female, J5 Conn_01x20_Female, Q1 BSS123, Q2 BSS123, Q3 BSS123, U1 4066, U2 LM386, U3 MCP6001U

Commit message: change board to radio connector
Parts:
- removed J2: Conn_01x06_Male, symbol Connector:Conn_01x06_Male
- added J2: DB9_Female, symbol Connector:DB9_Female
Connections:
- net labels added: Rx_AUD, Tx_AUD, Tx_OUT
- wire segments 162 -> 160
Other:
- note added: "To GM300 Connector"
- note removed: "GM300 connector"
Changed lines of the file:
@@
-$EndComp
-$Comp
-L Connector:Conn_01x06_Male J2
-U 1 1 603EE191
-P 950 5750
-F 0 "J2" H 1058 6131 50  0000 C CNN
-F 1 "Conn_01x06_Male" H 1058 6040 50  0000 C CNN
-F 2 "" H 950 5750 50  0001 C CNN
-F 3 "~" H 950 5750 50  0001 C CNN
-	1    950  5750
-	1    0    0    -1
 $EndComp
 $Comp
@@
 $EndComp
 $Comp
-L power:GND #PWR02
-U 1 1 603F2D64
-P 1350 6100
-F 0 "#PWR02" H 1350 5850 50  0001 C CNN
-F 1 "GND" H 1355 5927 50  0000 C CNN
-F 2 "" H 1350 6100 50  0001 C CNN
-F 3 "" H 1350 6100 50  0001 C CNN
-	1    1350 6100
-	1    0    0    -1
-$EndComp
-Wire Wire Line
-	1150 6050 1350 6050
-Wire Wire Line
-	1350 6050 1350 6100
-Wire Wire Line
-	1150 5950 1350 5950
-Wire Wire Line
-	1350 5950 1350 6050
-Connection ~ 1350 6050
-Wire Wire Line
-	1150 5850 1450 5850
-Wire Wire Line
-	1450 5750 1150 5750
-Wire Wire Line
-	1150 5550 1450 5550
-Wire Wire Line
-	1150 5650 1450 5650
-Text GLabel 1450 5850 2    50   Input ~ 0
-SPK_OUT
-Text GLabel 1450 5750 2    50   Input ~ 0
-RX_AUD
-Text GLabel 1450 5650 2    50   Input ~ 0
-TX_AUD
-$Comp
 L power:GND #PWR011
 U 1 1 60401F74
@@
 Text GLabel 4000 5150 2    50   Input ~ 0
 RX_AUD_INV
-Text GLabel 1450 5550 2    50   Input ~ 0
-TX_OUT
 $Comp
 L Device:C_Polarized C7
@@
 Volume
 Text Notes 750  5300 0    50   ~ 0
-GM300 connector
+To GM300 Connector
 Text Notes 700  3500 0    50   ~ 0
 To RPi USB soundcard
@@
 	7100 3800 7350 3800
 Connection ~ 7350 3800
+$Comp
+L Connector:DB9_Female J2
+U 1 1 603884B0
+P 1450 5950
+F 0 "J2" H 1630 5996 50  0000 L CNN
+F 1 "DB9_Female" H 1630 5905 50  0000 L CNN
+F 2 "" H 1450 5950 50  0001 C CNN
+F 3 " ~" H 1450 5950 50  0001 C CNN
+	1    1450 5950
+	1    0    0    -1
+$EndComp
+Text GLabel 950  5550 0    50   Input ~ 0
+Tx_OUT
+Text GLabel 950  5750 0    50   Input ~ 0
+Tx_AUD
+Text GLabel 950  5950 0    50   Input ~ 0
+Rx_AUD
+Text GLabel 950  6150 0    50   Input ~ 0
+SPK_OUT
+Text GLabel 1050 5650 0    50   Input ~ 0
+GND
+Text GLabel 1050 6250 0    50   Input ~ 0
+GND
+Wire Wire Line
+	1150 5550 950  5550
+Wire Wire Line
+	1150 5650 1050 5650
+Wire Wire Line
+	1150 5750 950  5750
+Wire Wire Line
+	1150 5950 950  5950
+Wire Wire Line
+	1150 6150 950  6150
+Wire Wire Line
+	1150 6250 1050 6250
 $EndSCHEMATC

Commit message: clean up a few erc warnings
Parts:
- gave numbers to parts that had none: 3
Connections:
- no-connect marks 0 -> 40
Changed lines of the file:
@@
 	1400 1850 1750 1850
-Wire Wire Line
-	1750 2400 1750 2500
 Wire Wire Line
 	1750 2100 1750 1850
@@
 Power supply\n12-15V
 $Comp
-L Connector:Conn_01x02_Female J?
+L Connector:Conn_01x02_Female J6
 U 1 1 6072C8C5
 P 900 7250
-F 0 "J?" H 792 6925 50  0000 C CNN
+F 0 "J6" H 792 6925 50  0000 C CNN
 F 1 "Conn_01x02_Female" H 792 7016 50  0000 C CNN
 F 2 "" H 900 7250 50  0001 C CNN
@@
 	1100 7150 1450 7150
 $Comp
-L Device:R R?
+L Device:R R14
 U 1 1 60753E7A
 P 8050 5000
-F 0 "R?" V 8257 5000 50  0000 C CNN
+F 0 "R14" V 8257 5000 50  0000 C CNN
 F 1 "39k" V 8166 5000 50  0000 C CNN
 F 2 "" V 7980 5000 50  0001 C CNN
@@
 	3950 6600 4100 6600
 $Comp
-L Device:R R?
+L Device:R R15
 U 1 1 607A773F
 P 2100 4200
-F 0 "R?" H 2031 4154 50  0000 R CNN
+F 0 "R15" H 2031 4154 50  0000 R CNN
 F 1 "100k" H 2031 4245 50  0000 R CNN
 F 2 "" V 2030 4200 50  0001 C CNN
@@
 	2100 4600 2100 4350
 $Comp
-L power:GND #PWR?
+L power:GND #PWR0101
 U 1 1 607C7423
 P 2100 4600
-F 0 "#PWR?" H 2100 4350 50  0001 C CNN
+F 0 "#PWR0101" H 2100 4350 50  0001 C CNN
 F 1 "GND" H 2105 4427 50  0000 C CNN
 F 2 "" H 2100 4600 50  0001 C CNN
@@
 Wire Wire Line
 	1150 6250 1050 6250
+NoConn ~ 1150 5850
+NoConn ~ 1150 6050
+NoConn ~ 1150 6350
+NoConn ~ 9100 1250
+NoConn ~ 9100 1450
+NoConn ~ 9100 1550
+NoConn ~ 9100 1650
+NoConn ~ 9100 1750
+NoConn ~ 9100 1850
+NoConn ~ 9100 1950
+NoConn ~ 9100 2050
+NoConn ~ 9100 2150
+NoConn ~ 9100 2250
+NoConn ~ 9100 2350
+NoConn ~ 9100 2450
+NoConn ~ 9100 2550
+NoConn ~ 9100 2650
+NoConn ~ 9100 2750
+NoConn ~ 9100 2850
+NoConn ~ 10400 2850
+NoConn ~ 10400 2750
+NoConn ~ 10400 2650
+NoConn ~ 10400 2550
+NoConn ~ 10400 2450
+NoConn ~ 10400 2350
+NoConn ~ 10400 2250
+NoConn ~ 10400 2150
+NoConn ~ 10400 2050
+NoConn ~ 10400 1950
+NoConn ~ 10400 1850
+NoConn ~ 10400 1750
+NoConn ~ 10400 1650
+NoConn ~ 10400 1450
+NoConn ~ 10400 1350
+NoConn ~ 10400 1250
+Wire Wire Line
+	1750 2400 1750 2500
+NoConn ~ 1400 1350
+NoConn ~ 1400 1450
+NoConn ~ 1400 1550
+NoConn ~ 1400 1950
+NoConn ~ 1400 2050
 $EndSCHEMATC

Commit message: fixin' labels
Connections:
- net Rx_AUD is gone; now on net RX_AUD: J2.3
- net Tx_AUD is gone; now on net TX_AUD: J2.2
- net Tx_OUT is gone; now on net TX_OUT: J2.1
Changed lines of the file:
@@
 $EndComp
 Text GLabel 950  5550 0    50   Input ~ 0
-Tx_OUT
+TX_OUT
 Text GLabel 950  5750 0    50   Input ~ 0
-Tx_AUD
+TX_AUD
 Text GLabel 950  5950 0    50   Input ~ 0
-Rx_AUD
+RX_AUD
 Text GLabel 950  6150 0    50   Input ~ 0
 SPK_OUT

Commit message: pushin' pushin' pushin'
Parts:
- J1: footprint (none) -> Connector_RJ:RJ45_Amphenol_RJHSE5380
Connections:
- no-connect marks 40 -> 43
Changed lines of the file:
@@
 F 0 "J1" H 1057 2417 50  0000 C CNN
 F 1 "RJ45" H 1057 2326 50  0000 C CNN
-F 2 "" V 1000 1775 50  0001 C CNN
+F 2 "Connector_RJ:RJ45_Amphenol_RJHSE5380" V 1000 1775 50  0001 C CNN
 F 3 "~" V 1000 1775 50  0001 C CNN
 	1    1000 1750
@@
 NoConn ~ 1400 1950
 NoConn ~ 1400 2050
+NoConn ~ 9150 5050
+NoConn ~ 9150 5650
+NoConn ~ 9250 5650
 $EndSCHEMATC

Commit message: some changes, bro. new pdf
Parts:
- added D?: LED, symbol Device:LED
- added R?: 2k2, symbol Device:R
- J1: symbol Connector:RJ45 -> Connector:8P8C
Connections:
- net +5V: now also U3.5 (V+)
- net +BATT: no longer U3.5 (V+)
- net GND: now also R?.2
- new net: D?.1 (K), R?.1
- new net ACT: D?.2 (A)
Other:
- moved on the sheet: D2, D3, R6, R7
Changed lines of the file:
@@
 L Device:R R7
 U 1 1 60384E06
-P 7800 1850
-F 0 "R7" H 7870 1896 50  0000 L CNN
-F 1 "1k" H 7870 1805 50  0000 L CNN
-F 2 "" V 7730 1850 50  0001 C CNN
-F 3 "~" H 7800 1850 50  0001 C CNN
-	1    7800 1850
+P 7550 1850
+F 0 "R7" H 7620 1896 50  0000 L CNN
+F 1 "1k" H 7620 1805 50  0000 L CNN
+F 2 "" V 7480 1850 50  0001 C CNN
+F 3 "~" H 7550 1850 50  0001 C CNN
+	1    7550 1850
 	1    0    0    -1
 $EndComp
@@
 	1400 1750 1650 1750
 $Comp
-L Connector:RJ45 J1
+L Connector:8P8C J1
 U 1 1 603919FB
 P 1000 1750
@@
 L Device:LED D3
 U 1 1 603B229A
-P 7800 1450
-F 0 "D3" V 7839 1332 50  0000 R CNN
-F 1 "RED" V 7748 1332 50  0000 R CNN
-F 2 "" H 7800 1450 50  0001 C CNN
-F 3 "~" H 7800 1450 50  0001 C CNN
-	1    7800 1450
+P 7550 1450
+F 0 "D3" V 7589 1332 50  0000 R CNN
+F 1 "RED" V 7498 1332 50  0000 R CNN
+F 2 "" H 7550 1450 50  0001 C CNN
+F 3 "~" H 7550 1450 50  0001 C CNN
+	1    7550 1450
 	0    -1   -1   0
 $EndComp
@@
 L Device:LED D2
 U 1 1 603C0CB1
-P 7450 1450
-F 0 "D2" V 7489 1332 50  0000 R CNN
-F 1 "GRN" V 7398 1332 50  0000 R CNN
-F 2 "" H 7450 1450 50  0001 C CNN
-F 3 "~" H 7450 1450 50  0001 C CNN
-	1    7450 1450
+P 7200 1450
+F 0 "D2" V 7239 1332 50  0000 R CNN
+F 1 "GRN" V 7148 1332 50  0000 R CNN
+F 2 "" H 7200 1450 50  0001 C CNN
+F 3 "~" H 7200 1450 50  0001 C CNN
+	1    7200 1450
 	0    -1   -1   0
 $EndComp
@@
 L Device:R R6
 U 1 1 603C168C
-P 7450 1850
-F 0 "R6" H 7520 1896 50  0000 L CNN
-F 1 "2k2" H 7520 1805 50  0000 L CNN
-F 2 "" V 7380 1850 50  0001 C CNN
-F 3 "~" H 7450 1850 50  0001 C CNN
-	1    7450 1850
+P 7200 1850
+F 0 "R6" H 7270 1896 50  0000 L CNN
+F 1 "2k2" H 7270 1805 50  0000 L CNN
+F 2 "" V 7130 1850 50  0001 C CNN
+F 3 "~" H 7200 1850 50  0001 C CNN
+	1    7200 1850
 	1    0    0    -1
 $EndComp
@@
 L power:+5V #PWR020
 U 1 1 603CAF2C
-P 7450 1200
-F 0 "#PWR020" H 7450 1050 50  0001 C CNN
-F 1 "+5V" H 7465 1373 50  0000 C CNN
-F 2 "" H 7450 1200 50  0001 C CNN
-F 3 "" H 7450 1200 50  0001 C CNN
-	1    7450 1200
+P 7200 1200
+F 0 "#PWR020" H 7200 1050 50  0001 C CNN
+F 1 "+5V" H 7215 1373 50  0000 C CNN
+F 2 "" H 7200 1200 50  0001 C CNN
+F 3 "" H 7200 1200 50  0001 C CNN
+	1    7200 1200
 	1    0    0    -1
 $EndComp
@@
 L power:GND #PWR021
 U 1 1 603CB60E
-P 7450 2100
-F 0 "#PWR021" H 7450 1850 50  0001 C CNN
-F 1 "GND" H 7455 1927 50  0000 C CNN
-F 2 "" H 7450 2100 50  0001 C CNN
-F 3 "" H 7450 2100 50  0001 C CNN
-	1    7450 2100
+P 7200 2100
+F 0 "#PWR021" H 7200 1850 50  0001 C CNN
+F 1 "GND" H 7205 1927 50  0000 C CNN
+F 2 "" H 7200 2100 50  0001 C CNN
+F 3 "" H 7200 2100 50  0001 C CNN
+	1    7200 2100
 	1    0    0    -1
 $EndComp
@@
 L power:GND #PWR022
 U 1 1 603CBEBC
-P 7800 2100
-F 0 "#PWR022" H 7800 1850 50  0001 C CNN
-F 1 "GND" H 7805 1927 50  0000 C CNN
-F 2 "" H 7800 2100 50  0001 C CNN
-F 3 "" H 7800 2100 50  0001 C CNN
-	1    7800 2100
-	1    0    0    -1
-$EndComp
-Wire Wire Line
-	7800 1200 7800 1300
-Wire Wire Line
-	7450 2100 7450 2000
-Wire Wire Line
-	7450 1200 7450 1300
-Wire Wire Line
-	7450 1600 7450 1700
-Wire Wire Line
-	7800 1600 7800 1700
-Wire Wire Line
-	7800 2000 7800 2100
-Text GLabel 7800 1200 1    50   Input ~ 0
+P 7550 2100
+F 0 "#PWR022" H 7550 1850 50  0001 C CNN
+F 1 "GND" H 7555 1927 50  0000 C CNN
+F 2 "" H 7550 2100 50  0001 C CNN
+F 3 "" H 7550 2100 50  0001 C CNN
+	1    7550 2100
+	1    0    0    -1
+$EndComp
+Wire Wire Line
+	7550 1200 7550 1300
+Wire Wire Line
+	7200 2100 7200 2000
+Wire Wire Line
+	7200 1200 7200 1300
+Wire Wire Line
+	7200 1600 7200 1700
+Wire Wire Line
+	7550 1600 7550 1700
+Wire Wire Line
+	7550 2000 7550 2100
+Text GLabel 7550 1200 1    50   Input ~ 0
 TX_EN
 $Comp
@@
 Text Notes 9700 1900 0    50   ~ 0
 RPi
-Text Notes 8000 1650 0    50   ~ 0
+Text Notes 7750 1650 0    50   ~ 0
 TX
-Text Notes 7200 1650 0    50   ~ 0
+Text Notes 6950 1650 0    50   ~ 0
 PWR
 $Comp
@@
 Wire Wire Line
 	4300 7000 4300 7050
-Wire Wire Line
-	4300 6350 4300 6400
 $Comp
 L Device:R R10
@@
 Wire Wire Line
 	4850 6700 4850 7300
-$Comp
-L power:+BATT #PWR037
-U 1 1 60631654
-P 4300 6350
-F 0 "#PWR037" H 4300 6200 50  0001 C CNN
-F 1 "+BATT" V 4315 6477 50  0000 L CNN
-F 2 "" H 4300 6350 50  0001 C CNN
-F 3 "" H 4300 6350 50  0001 C CNN
-	1    4300 6350
-	1    0    0    -1
-$EndComp
 $Comp
 L Device:R R11
@@
 NoConn ~ 9150 5650
 NoConn ~ 9250 5650
+$Comp
+L Device:LED D?
+U 1 1 605F2274
+P 7900 1450
+F 0 "D?" V 7939 1332 50  0000 R CNN
+F 1 "LED" V 7848 1332 50  0000 R CNN
+F 2 "" H 7900 1450 50  0001 C CNN
+F 3 "~" H 7900 1450 50  0001 C CNN
+	1    7900 1450
+	0    -1   -1   0
+$EndComp
+Text GLabel 7900 1200 1    50   Input ~ 0
+ACT
+Wire Wire Line
+	7900 1200 7900 1300
+$Comp
+L Device:R R?
+U 1 1 605FD1E2
+P 7900 1850
+F 0 "R?" H 7970 1896 50  0000 L CNN
+F 1 "2k2" H 7970 1805 50  0000 L CNN
+F 2 "" V 7830 1850 50  0001 C CNN
+F 3 "~" H 7900 1850 50  0001 C CNN
+	1    7900 1850
+	1    0    0    -1
+$EndComp
+Wire Wire Line
+	7900 1600 7900 1700
+$Comp
+L power:GND #PWR?
+U 1 1 6060746D
+P 7900 2100
+F 0 "#PWR?" H 7900 1850 50  0001 C CNN
+F 1 "GND" H 7905 1927 50  0000 C CNN
+F 2 "" H 7900 2100 50  0001 C CNN
+F 3 "" H 7900 2100 50  0001 C CNN
+	1    7900 2100
+	1    0    0    -1
+$EndComp
+Wire Wire Line
+	7900 2000 7900 2100
+$Comp
+L power:+5V #PWR?
+U 1 1 6061B443
+P 4300 6250
+F 0 "#PWR?" H 4300 6100 50  0001 C CNN
+F 1 "+5V" H 4315 6423 50  0000 C CNN
+F 2 "" H 4300 6250 50  0001 C CNN
+F 3 "" H 4300 6250 50  0001 C CNN
+	1    4300 6250
+	1    0    0    -1
+$EndComp
+Wire Wire Line
+	4300 6250 4300 6400
 $EndSCHEMATC

Commit message: sync
Connections:
- net +5V: now also R12.2, R9.2
- net +BATT: no longer R12.2, R9.2
- net ACT: now also J4.15 (Pin_15)
- no-connect marks 43 -> 42
Changed lines of the file:
@@
-$EndComp
-$Comp
-L Connector:Conn_01x20_Female J4
-U 1 1 60387CF1
-P 9300 1850
-F 0 "J4" H 9150 800 50  0000 L CNN
-F 1 "Conn_01x20_Female" H 8800 700 50  0000 L CNN
-F 2 "" H 9300 1850 50  0001 C CNN
-F 3 "~" H 9300 1850 50  0001 C CNN
-	1    9300 1850
-	1    0    0    -1
 $EndComp
 $Comp
@@
 	-1   0    0    1
 $EndComp
-$Comp
-L power:+BATT #PWR036
-U 1 1 60678A85
-P 3950 6000
-F 0 "#PWR036" H 3950 5850 50  0001 C CNN
-F 1 "+BATT" V 3965 6127 50  0000 L CNN
-F 2 "" H 3950 6000 50  0001 C CNN
-F 3 "" H 3950 6000 50  0001 C CNN
-	1    3950 6000
-	1    0    0    -1
-$EndComp
 Text GLabel 2900 6800 0    50   Input ~ 0
 RX_AUD
@@
 	1    2750 6000
 	-1   0    0    1
-$EndComp
-$Comp
-L power:+BATT #PWR033
-U 1 1 606A9F0E
-P 3000 6000
-F 0 "#PWR033" H 3000 5850 50  0001 C CNN
-F 1 "+BATT" V 3015 6127 50  0000 L CNN
-F 2 "" H 3000 6000 50  0001 C CNN
-F 3 "" H 3000 6000 50  0001 C CNN
-	1    3000 6000
-	1    0    0    -1
 $EndComp
 Wire Wire Line
@@
 NoConn ~ 9100 2150
 NoConn ~ 9100 2250
-NoConn ~ 9100 2350
 NoConn ~ 9100 2450
 NoConn ~ 9100 2550
@@
 	7900 1600 7900 1700
 $Comp
-L power:GND #PWR?
+L power:GND #PWR0102
 U 1 1 6060746D
 P 7900 2100
-F 0 "#PWR?" H 7900 1850 50  0001 C CNN
+F 0 "#PWR0102" H 7900 1850 50  0001 C CNN
 F 1 "GND" H 7905 1927 50  0000 C CNN
 F 2 "" H 7900 2100 50  0001 C CNN
@@
 	7900 2000 7900 2100
 $Comp
-L power:+5V #PWR?
+L power:+5V #PWR0103
 U 1 1 6061B443
 P 4300 6250
-F 0 "#PWR?" H 4300 6100 50  0001 C CNN
+F 0 "#PWR0103" H 4300 6100 50  0001 C CNN
 F 1 "+5V" H 4315 6423 50  0000 C CNN
 F 2 "" H 4300 6250 50  0001 C CNN
@@
 Wire Wire Line
 	4300 6250 4300 6400
+$Comp
+L power:+5V #PWR?
+U 1 1 6062EAEF
+P 3000 6000
+F 0 "#PWR?" H 3000 5850 50  0001 C CNN
+F 1 "+5V" H 3015 6173 50  0000 C CNN
+F 2 "" H 3000 6000 50  0001 C CNN
+F 3 "" H 3000 6000 50  0001 C CNN
+	1    3000 6000
+	1    0    0    -1
+$EndComp
+$Comp
+L power:+5V #PWR?
+U 1 1 6062F1B2
+P 3950 6000
+F 0 "#PWR?" H 3950 5850 50  0001 C CNN
+F 1 "+5V" H 3965 6173 50  0000 C CNN
+F 2 "" H 3950 6000 50  0001 C CNN
+F 3 "" H 3950 6000 50  0001 C CNN
+	1    3950 6000
+	1    0    0    -1
+$EndComp
+Text GLabel 8800 2350 0    50   Input ~ 0
+ACT
+Wire Wire Line
+	9100 2350 8800 2350
+$Comp
+L Connector:Conn_01x20_Female J4
+U 1 1 60387CF1
+P 9300 1850
+F 0 "J4" H 9150 800 50  0000 L CNN
+F 1 "Conn_01x20_Female" H 8800 700 50  0000 L CNN
+F 2 "" H 9300 1850 50  0001 C CNN
+F 3 "~" H 9300 1850 50  0001 C CNN
+	1    9300 1850
+	1    0    0    -1
+$EndComp
 $EndSCHEMATC

Commit message: redraw
Parts:
- removed C5: 100u/16V, symbol Device:C_Polarized
- removed C6: 470n, symbol Device:C
- removed C7: 220u/35V, symbol Device:C_Polarized
- removed C8, C9: 220n, symbol Device:C
- removed D1: 3V3, symbol Device:D_Zener
- removed D?: LED, symbol Device:LED
- removed J1: RJ45, Connector_RJ:RJ45_Amphenol_RJHSE5380, symbol Connector:8P8C
- removed J2: DB9_Female, symbol Connector:DB9_Female
- removed J3: RPi_SND, symbol Connector:AudioJack3
- removed J4, J5: Conn_01x20_Female, symbol Connector:Conn_01x20_Female
- removed J6: Conn_01x02_Female, symbol Connector:Conn_01x02_Female
- removed Q1, Q2, Q3: BSS123, Package_TO_SOT_SMD:SOT-23, symbol Transistor_FET:BSS123
- removed R10, R13: 10k, symbol Device:R
- removed R11, R12, R9: 22k, symbol Device:R
- removed R14: 39k, symbol Device:R
- removed R15: 100k, symbol Device:R
- removed R?: 2k2, symbol Device:R
- removed RV3: 4k7, symbol Device:R_Potentiometer
- removed U3: MCP6001U, symbol Amplifier_Operational:MCP6001U
- added C5: 470n, Capacitor_THT:C_Disc_D5.0mm_W2.5mm_P5.00mm, symbol Device:C
- added D1: BLU, LED_THT:LED_D3.0mm, symbol Device:LED
- added J1: RPi Header, Connector_PinSocket_2.54mm:PinSocket_2x20_P2.54mm_Vertical, symbol Connector_Generic:Conn_02x20_Odd_Even
- added J2: 1935161, PHOENIX_1935161, symbol 1935161:1935161
- added J3: DB9_Female, Connector_Dsub:DSUB-9_Female_Horizontal_P2.77x2.84mm_EdgePinOffset4.94mm_Housed_MountingHolesOffset7.48mm, symbol Connector:DB9_Female
- added J4: RJ45, Connector_RJ:RJ45_Amphenol_54602-x08_Horizontal, symbol Connector:RJ45
- added J5: SJ1-3523N, CUI_SJ1-3523N, symbol SJ1-3523N:SJ1-3523N
- added Q1, Q2, Q3: 2N7000, Package_TO_SOT_THT:TO-92_HandSolder, symbol Transistor_FET:2N7000
- added R? (x2): 47K, Resistor_THT:R_Axial_DIN0207_L6.3mm_D2.5mm_P7.62mm_Horizontal, symbol Device:R
- added SW?: SW_Push, symbol Switch:SW_Push
- C1: value 22u/25V -> 22u; footprint (none) -> Capacitor_THT:CP_Radial_D8.0mm_P5.00mm
- C2: footprint (none) -> Capacitor_THT:C_Disc_D5.0mm_W2.5mm_P5.00mm
- C3: value 47u/25V -> 47u; footprint (none) -> Capacitor_THT:CP_Radial_D8.0mm_P5.00mm
- C4: value 100u/25V -> 220u; footprint (none) -> Capacitor_THT:CP_Radial_D8.0mm_P5.00mm
- D2: value GRN -> RED; footprint (none) -> LED_THT:LED_D3.0mm
- D3: value RED -> GRN; footprint (none) -> LED_THT:LED_D3.0mm
- R1: value 390R -> 2K2; footprint (none) -> Resistor_THT:R_Axial_DIN0207_L6.3mm_D2.5mm_P7.62mm_Horizontal
- R2: value 680R -> 1K; footprint (none) -> Resistor_THT:R_Axial_DIN0207_L6.3mm_D2.5mm_P7.62mm_Horizontal
- R3: value 39k -> 2K2; footprint (none) -> Resistor_THT:R_Axial_DIN0207_L6.3mm_D2.5mm_P7.62mm_Horizontal
- R4: value 47k -> 390R; footprint (none) -> Resistor_THT:R_Axial_DIN0207_L6.3mm_D2.5mm_P7.62mm_Horizontal
- R5: value 47k -> 680R; footprint (none) -> Resistor_THT:R_Axial_DIN0207_L6.3mm_D2.5mm_P7.62mm_Horizontal
- R6: value 2k2 -> 100K; footprint (none) -> Resistor_THT:R_Axial_DIN0207_L6.3mm_D2.5mm_P7.62mm_Horizontal
- R7: value 1k -> 22K; footprint (none) -> Resistor_THT:R_Axial_DIN0207_L6.3mm_D2.5mm_P7.62mm_Horizontal
- R8: value 22k -> 39K; footprint (none) -> Resistor_THT:R_Axial_DIN0207_L6.3mm_D2.5mm_P7.62mm_Horizontal
- RV1: value 4k7 -> 4K7
- RV2: value 1k -> 1K
Connections:
- net +3V3: now also R7.1, J1.1 (Pin_1)
- net +5V: now also D1.2 (A), J1.2 (Pin_2); no longer D2.2 (A)
- net +BATT: now also J2.2, R?.1, R?.1; no longer C4.1, R2.1, R4.1
- net ACT: now also D3.2 (A), J1.29 (Pin_29)
- net GND: now also R1.2, R2.2, R3.2, J1.14 (Pin_14), J1.30 (Pin_30), J1.34 (Pin_34), J1.39 (Pin_39), J1.6 (Pin_6), J1.9 (Pin_9), J2.1, J3.6, J3.9, J4.5, J5.1, Q1.1 (S), Q2.1 (S), Q3.1 (S), SW?.2; no longer C4.2, R7.2, R8.2, U2.2 (-)
- net MIC: now also R4.2, J4.4; no longer R1.2
- net PTT: now also J1.3 (Pin_3), J4.3
- net RX_AUD: now also J3.3; no longer R8.1
- net RX_AUD_INV: no longer RV1.2
- net SPK_AMP: now also R8.2, U1.8; no longer U1.9
- net SPK_OUT: now also C4.2, J3.4
- net TX_AUD: now also J3.2
- net TX_EN: now also D2.2 (A), J1.5 (Pin_5), Q2.2 (G), Q3.2 (G); no longer D3.2 (A)
- net TX_OUT: now also J3.1, Q3.3 (D)
- net at U1.1: now also U1.9, J5.2; no longer U1.8
- net at C2.1, D4.1 (K), U1.4: now also R6.1, J5.3
- net at R3.1: now also D3.1 (K); no longer RV1.3
- net at U2.3 (+): now also C5.1
- net at U2.5: now also C4.1
- net at D2.1 (K): now also R2.1; no longer R6.1
- net SW_1 renamed SW1
- net SW1: now also Q1.3 (D), R?.2; no longer R4.2
- net SW_2 renamed SW2
- net SW2: now also Q1.2 (G), Q2.3 (D), R?.2; no longer R5.2
- new net: D1.1 (K), R1.1
- new net: C1.1, R4.1, R5.2
- new net: C5.2, RV1.2
- new net: R8.1, RV1.3
- new net PWR_DOWN: J1.7 (Pin_7), R7.2, SW?.1
- no-connect marks 42 -> 0
Other:
- note added: "Connector To Radio"
- note added: "Indicator LEDs"
- note added: "Microphone Connector"
- note added: "Power In"
- note added: "Power Supply\n12v - 15v"
- note added: "RPi Audio In / Out"
- note added: "RPi Header"
- note added: "RPi Shutdown"
- note added: "TX FM Deviation"
- note removed: "Add a DC/DC converter"
- note removed: "Check the connections!"
- note removed: "HMN 1035C"
- note removed: "PWR"
- note removed: "Power supply\n12-15V"
- note removed: "RPi"
- note removed: "Received baseband\nsignal level"
- note removed: "TX"
- note removed: "TX FM deviation"
- note removed: "TX:\nSW_1 - H\nSW_2 - L\n\nRX:\nSW_1 - L\nSW_2 - H"
- note removed: "TX_EN:\nTX - H\nRX - L"
- note removed: "TX_OUT has to be pulled\nto GND for TX"
- note removed: "To GM300 Connector"
- note removed: "To RPi USB soundcard"

Commit message: little things
Parts:
- C1, C3, C4: symbol Device:C_Polarized -> M17_GM300_RPi-rescue:C_Polarized-Device
- RV1, RV2: symbol Device:R_Potentiometer -> M17_GM300_RPi-rescue:R_Potentiometer-Device
Connections:
- net +5V: now also J1.4 (Pin_4)
- no-connect marks 0 -> 27
Other:
- note added: "TRX Switch"
- note added: "TX_EN\nTX - H\nRX - L"
- note added: "TX_OUT is pulled\nto GND for TX"
