File: M17_GM300_RPi.sch (KiCad schematic (older format))
At the start: 33 parts, among them J1 RPi Header, J2 1935161, J3 DB9_Female, J4 RJ45, J5 SJ1-3523N, Q1 2N7000, Q2 2N7000, Q3 2N7000, U1 4066, U2 LM386

Commit message: draft alpha
Parts:
- added C6, C7: 220n, Capacitor_THT:C_Disc_D5.0mm_W2.5mm_P5.00mm, symbol Device:C
- added C8: 10u Tantalum, symbol Device:CP
- added C9: 2.0u Tantalum, symbol Device:CP
- added R11: 39K, Resistor_THT:R_Axial_DIN0207_L6.3mm_D2.5mm_P7.62mm_Horizontal, symbol Device:R
- added R12, R13: 10K, Resistor_THT:R_Axial_DIN0207_L6.3mm_D2.5mm_P7.62mm_Horizontal, symbol Device:R
- added R14, R15, R16, R17: 22K, Resistor_THT:R_Axial_DIN0207_L6.3mm_D2.5mm_P7.62mm_Horizontal, symbol Device:R
- added RV3: R_POT, symbol Device:R_POT
- added U3: MCP6002-I/P, symbol Amplifier_Operational:MCP6002-xP
- added U4: LT323AT-PBF, TO220-3_T_LIT, symbol 2021-02-26_21-39-49:LT323AT-PBF
- gave numbers to parts that had none: 3
Connections:
- net labels added: 2V5
- wire segments 102 -> 136
- no-connect marks 27 -> 38
Other:
- note added: "Power Regulator"
- note added: "RX Baseband Signal Level"

Commit message: Add files via upload
Parts:
- removed C6, C7: 220n, Capacitor_THT:C_Disc_D5.0mm_W2.5mm_P5.00mm, symbol Device:C
- removed R6: 100K, Resistor_THT:R_Axial_DIN0207_L6.3mm_D2.5mm_P7.62mm_Horizontal, symbol Device:R
- added C6, C7: 10u, Capacitor_THT:CP_Radial_D8.0mm_P5.00mm, symbol M17_GM300_RPi-rescue:C_Polarized-Device
- R11: value 39K -> 100R
- R12: value 10K -> 22K
- R14, R16: value 22K -> 10K
- R15: value 22K -> 33K
- RV3: value R_POT -> 4K7
Connections:
- net labels removed: 2V5
- wire segments 136 -> 141
Other:
- note added: "MAX7413CPE+ goes here"
- note added: "replace me with a SMPS"
- moved on the sheet: R11, R13, R16, R17, R7, SW1, U3A, U3B, U3C

Commit message: it aint pretty.
Parts:
- C8, C9: symbol Device:CP -> M17_GM300_RPi-rescue:CP-Device
- RV3: symbol Device:R_POT -> M17_GM300_RPi-rescue:R_POT-Device
Connections:
- net labels added: FLT_CLK
- no-connect marks 38 -> 37
Changed lines of the file:
@@
 $Descr A4 11693 8268
 encoding utf-8
-Sheet 1 1
+Sheet 1 2
 Title "M17 Radio Interface for Motorola GM300 Radio"
 Date "2021-02-26"
@@
 	10750 1050 10900 1050
 Wire Wire Line
-	10900 1050 10900 1450
-Wire Wire Line
 	10750 1450 10900 1450
-Connection ~ 10900 1450
 Wire Wire Line
 	10900 1450 10900 2250
@@
 NoConn ~ 10750 1650
 NoConn ~ 10750 1550
-NoConn ~ 10750 1350
 NoConn ~ 10750 1250
 NoConn ~ 10750 1150
@@
 	1350 1450 1200 1450
 $Comp
-L Device:CP C9
+L M17_GM300_RPi-rescue:CP-Device C9
 U 1 1 604E346D
 P 1200 1800
@@
 $EndComp
 $Comp
-L Device:CP C8
+L M17_GM300_RPi-rescue:CP-Device C8
 U 1 1 604E358D
 P 3700 1800
@@
 $EndComp
 $Comp
-L Device:R_POT RV3
+L M17_GM300_RPi-rescue:R_POT-Device RV3
 U 1 1 605542C0
 P 4600 4900
@@
 Wire Wire Line
 	7650 3800 8250 3800
+$Comp
+L power:GND #PWR?
+U 1 1 60533649
+P 10900 1050
+F 0 "#PWR?" H 10900 800 50  0001 C CNN
+F 1 "GND" V 10905 922 50  0000 R CNN
+F 2 "" H 10900 1050 50  0001 C CNN
+F 3 "" H 10900 1050 50  0001 C CNN
+	1    10900 1050
+	0    -1   -1   0
+$EndComp
+Text GLabel 10850 1350 2    50   Input ~ 0
+FLT_CLK
+Wire Wire Line
+	10750 1350 10850 1350
+$Sheet
+S 1850 5950 900  500
+U 60549FFC
+F0 "M17 RX Baseband" 50
+F1 "RXBaseband.sch" 50
+$EndSheet
 $EndSCHEMATC

Commit message: Add files via upload
Parts:
- removed C6, C7: 10u, Capacitor_THT:CP_Radial_D8.0mm_P5.00mm, symbol M17_GM300_RPi-rescue:C_Polarized-Device
- removed D5: 2V7, symbol Device:D_Zener
- removed R11: 100R, Resistor_THT:R_Axial_DIN0207_L6.3mm_D2.5mm_P7.62mm_Horizontal, symbol Device:R
- removed R12, R17: 22K, Resistor_THT:R_Axial_DIN0207_L6.3mm_D2.5mm_P7.62mm_Horizontal, symbol Device:R
- removed R13, R14, R16: 10K, Resistor_THT:R_Axial_DIN0207_L6.3mm_D2.5mm_P7.62mm_Horizontal, symbol Device:R
- removed R15: 33K, Resistor_THT:R_Axial_DIN0207_L6.3mm_D2.5mm_P7.62mm_Horizontal, symbol Device:R
- removed RV3: 4K7, symbol M17_GM300_RPi-rescue:R_POT-Device
- removed U3: MCP6002-I/P, symbol Amplifier_Operational:MCP6002-xP
- added Q2: 2N7000, Package_TO_SOT_THT:TO-92_HandSolder, symbol Transistor_FET:2N7000
- renumbered C9 to C1, C8 to C2, C1 to C3, C2 to C4, C4 to C6, C3 to C7, D4 to D1, D1 to D2, D2 to D3, D3 to D4, J4 to J1, J5 to J2, J2 to J3, J3 to J4, J1 to J5, Q2 to Q3, Q3 to Q4, R10 to R1, R9 to R2, R4 to R3, R5 to R4, R8 to R5, R1 to R6, R2 to R7, R3 to R8, R7 to R9, RV2 to RV1, RV1 to RV2, U4 to U1, U1 to U2, U2 to U3
Connections:
- net labels added: MUTE, SPK_MUTE
- wire segments 141 -> 115
- no-connect marks 37 -> 36
Other:
- note removed: "MAX7413CPE+ goes here"
- moved on the sheet: D1, R5, RV2

Commit message: smps
Parts:
- removed C1: 2.0u Tantalum, symbol M17_GM300_RPi-rescue:CP-Device
- removed C2: 10u Tantalum, symbol M17_GM300_RPi-rescue:CP-Device
- removed U1: LT323AT-PBF, TO220-3_T_LIT, symbol 2021-02-26_21-39-49:LT323AT-PBF
- added C?: 100 uF, symbol Device:C_Polarized
- added C?: 1000 uF, symbol Device:C_Polarized
- added D?: V3PM6, symbol Device:D_Schottky
- added L?: 100 uH, symbol Device:L
- added U?: LM2576HVS-5, Package_TO_SOT_SMD:TO-263-5_TabPin3, symbol Regulator_Switching:LM2576HVS-5
Connections:
- wire segments 115 -> 125
Other:
- note removed: "replace me with a SMPS"
Changed lines of the file:
@@
 NoConn ~ 10750 1250
 NoConn ~ 10750 1150
-$Comp
-L power:+BATT #PWR01
-U 1 1 604D0679
-P 1000 1450
-F 0 "#PWR01" H 1000 1300 50  0001 C CNN
-F 1 "+BATT" V 1015 1577 50  0000 L CNN
-F 2 "" H 1000 1450 50  0001 C CNN
-F 3 "" H 1000 1450 50  0001 C CNN
-	1    1000 1450
-	0    -1   -1   0
-$EndComp
-$Comp
-L power:+5V #PWR05
-U 1 1 604D0FC4
-P 3950 1450
-F 0 "#PWR05" H 3950 1300 50  0001 C CNN
-F 1 "+5V" V 3965 1578 50  0000 L CNN
-F 2 "" H 3950 1450 50  0001 C CNN
-F 3 "" H 3950 1450 50  0001 C CNN
-	1    3950 1450
-	0    1    1    0
-$EndComp
-$Comp
-L 2021-02-26_21-39-49:LT323AT-PBF U1
-U 1 1 604D6162
-P 1350 1450
-F 0 "U1" H 2450 1837 60  0000 C CNN
-F 1 "LT323AT-PBF" H 2450 1731 60  0000 C CNN
-F 2 "TO220-3_T_LIT" H 2450 1690 60  0001 C CNN
-F 3 "" H 1350 1450 60  0000 C CNN
-	1    1350 1450
-	1    0    0    -1
-$EndComp
-$Comp
-L power:GND #PWR03
-U 1 1 604D700A
-P 2450 2150
-F 0 "#PWR03" H 2450 1900 50  0001 C CNN
-F 1 "GND" H 2455 1977 50  0000 C CNN
-F 2 "" H 2450 2150 50  0001 C CNN
-F 3 "" H 2450 2150 50  0001 C CNN
-	1    2450 2150
-	1    0    0    -1
-$EndComp
-Wire Wire Line
-	2450 2050 2450 2150
-Wire Wire Line
-	3550 1450 3700 1450
-Wire Wire Line
-	1350 1450 1200 1450
-$Comp
-L M17_GM300_RPi-rescue:CP-Device C1
-U 1 1 604E346D
-P 1200 1800
-F 0 "C1" H 1318 1846 50  0000 L CNN
-F 1 "2.0u Tantalum" H 1318 1755 50  0000 L CNN
-F 2 "" H 1238 1650 50  0001 C CNN
-F 3 "~" H 1200 1800 50  0001 C CNN
-	1    1200 1800
-	1    0    0    -1
-$EndComp
-$Comp
-L M17_GM300_RPi-rescue:CP-Device C2
-U 1 1 604E358D
-P 3700 1800
-F 0 "C2" H 3818 1846 50  0000 L CNN
-F 1 "10u Tantalum" H 3818 1755 50  0000 L CNN
-F 2 "" H 3738 1650 50  0001 C CNN
-F 3 "~" H 3700 1800 50  0001 C CNN
-	1    3700 1800
-	1    0    0    -1
-$EndComp
-$Comp
-L power:GND #PWR04
-U 1 1 604E3DE7
-P 3700 1950
-F 0 "#PWR04" H 3700 1700 50  0001 C CNN
-F 1 "GND" H 3705 1777 50  0000 C CNN
-F 2 "" H 3700 1950 50  0001 C CNN
-F 3 "" H 3700 1950 50  0001 C CNN
-	1    3700 1950
-	1    0    0    -1
-$EndComp
-$Comp
-L power:GND #PWR02
-U 1 1 604E4632
-P 1200 1950
-F 0 "#PWR02" H 1200 1700 50  0001 C CNN
-F 1 "GND" H 1205 1777 50  0000 C CNN
-F 2 "" H 1200 1950 50  0001 C CNN
-F 3 "" H 1200 1950 50  0001 C CNN
-	1    1200 1950
-	1    0    0    -1
-$EndComp
-Wire Wire Line
-	3700 1650 3700 1450
-Connection ~ 3700 1450
-Wire Wire Line
-	3700 1450 3950 1450
-Connection ~ 1200 1450
-Wire Wire Line
-	1200 1450 1000 1450
-Wire Wire Line
-	1200 1450 1200 1650
 Wire Notes Line
 	500  2900 11200 2900
@@
 Wire Wire Line
 	10550 5850 10550 5900
-Text Notes 1950 1450 0    50   ~ 0
-replace me with a SMPS
 $Comp
 L power:GND #PWR037
@@
 Text GLabel 4900 3750 1    50   Input ~ 0
 SPK_MUTE
+$Comp
+L Regulator_Switching:LM2576HVS-5 U?
+U 1 1 60542727
+P 2500 1400
+F 0 "U?" H 2500 1767 50  0000 C CNN
+F 1 "LM2576HVS-5" H 2500 1676 50  0000 C CNN
+F 2 "Package_TO_SOT_SMD:TO-263-5_TabPin3" H 2500 1150 50  0001 L CIN
+F 3 "http://www.ti.com/lit/ds/symlink/lm2576.pdf" H 2500 1400 50  0001 C CNN
+	1    2500 1400
+	1    0    0    -1
+$EndComp
+$Comp
+L power:+BATT #PWR?
+U 1 1 60543972
+P 1400 1300
+F 0 "#PWR?" H 1400 1150 50  0001 C CNN
+F 1 "+BATT" V 1415 1427 50  0000 L CNN
+F 2 "" H 1400 1300 50  0001 C CNN
+F 3 "" H 1400 1300 50  0001 C CNN
+	1    1400 1300
+	0    -1   -1   0
+$EndComp
+$Comp
+L power:GND #PWR?
+U 1 1 60543DCC
+P 2500 2000
+F 0 "#PWR?" H 2500 1750 50  0001 C CNN
+F 1 "GND" H 2505 1827 50  0000 C CNN
+F 2 "" H 2500 2000 50  0001 C CNN
+F 3 "" H 2500 2000 50  0001 C CNN
+	1    2500 2000
+	1    0    0    -1
+$EndComp
+$Comp
+L power:GND #PWR?
+U 1 1 605442BC
+P 1950 1650
+F 0 "#PWR?" H 1950 1400 50  0001 C CNN
+F 1 "GND" H 1955 1477 50  0000 C CNN
+F 2 "" H 1950 1650 50  0001 C CNN
+F 3 "" H 1950 1650 50  0001 C CNN
+	1    1950 1650
+	1    0    0    -1
+$EndComp
+Wire Wire Line
+	2000 1500 1950 1500
+Wire Wire Line
+	1950 1500 1950 1650
+Wire Wire Line
+	2500 1700 2500 2000
+$Comp
+L Device:C_Polarized C?
+U 1 1 6054C3EF
+P 1600 1600
+F 0 "C?" H 1718 1646 50  0000 L CNN
+F 1 "100 uF" H 1718 1555 50  0000 L CNN
+F 2 "" H 1638 1450 50  0001 C CNN
+F 3 "~" H 1600 1600 50  0001 C CNN
+	1    1600 1600
+	1    0    0    -1
+$EndComp
+$Comp
+L Device:L L?
+U 1 1 6054CA01
+P 3300 1500
+F 0 "L?" V 3490 1500 50  0000 C CNN
+F 1 "100 uH" V 3399 1500 50  0000 C CNN
+F 2 "" H 3300 1500 50  0001 C CNN
+F 3 "~" H 3300 1500 50  0001 C CNN
+	1    3300 1500
+	0    -1   -1   0
+$EndComp
+$Comp
+L Device:C_Polarized C?
+U 1 1 6054D08D
+P 3450 1650
+F 0 "C?" H 3568 1696 50  0000 L CNN
+F 1 "1000 uF" H 3568 1605 50  0000 L CNN
+F 2 "" H 3488 1500 50  0001 C CNN
+F 3 "~" H 3450 1650 50  0001 C CNN
+	1    3450 1650
+	1    0    0    -1
+$EndComp
+$Comp
+L power:+5V #PWR?
+U 1 1 6054D592
+P 3700 1500
+F 0 "#PWR?" H 3700 1350 50  0001 C CNN
+F 1 "+5V" V 3715 1628 50  0000 L CNN
+F 2 "" H 3700 1500 50  0001 C CNN
+F 3 "" H 3700 1500 50  0001 C CNN
+	1    3700 1500
+	0    1    1    0
+$EndComp
+Wire Wire Line
+	3000 1300 3700 1300
+Wire Wire Line
+	3700 1300 3700 1500
+Connection ~ 2500 2000
+Wire Wire Line
+	3100 2000 2500 2000
+Wire Wire Line
+	3450 1500 3700 1500
+Connection ~ 3450 1500
+Connection ~ 3700 1500
+Wire Wire Line
+	1600 1750 1600 2000
+Wire Wire Line
+	1600 2000 2500 2000
+Wire Wire Line
+	1400 1300 1600 1300
+Wire Wire Line
+	1600 1300 1600 1450
+Connection ~ 1600 1300
+Wire Wire Line
+	1600 1300 2000 1300
+$Comp
+L Device:D_Schottky D?
+U 1 1 6055A4E3
+P 3100 1850
+F 0 "D?" V 3054 1930 50  0000 L CNN
+F 1 "V3PM6" V 3145 1930 50  0000 L CNN
+F 2 "" H 3100 1850 50  0001 C CNN
+F 3 "~" H 3100 1850 50  0001 C CNN
+	1    3100 1850
+	0    1    1    0
+$EndComp
+Wire Wire Line
+	3000 1500 3100 1500
+Wire Wire Line
+	3100 1700 3100 1500
+Connection ~ 3100 1500
+Wire Wire Line
+	3100 1500 3150 1500
+Wire Wire Line
+	3450 1800 3450 2000
+Wire Wire Line
+	3450 2000 3100 2000
+Connection ~ 3100 2000
 $EndSCHEMATC

Commit message: change footprints to smd where aplicable
Parts:
- C1, C2: renamed from C?; footprint (none) -> Capacitor_SMD:C_0402_1005Metric; symbol Device:C_Polarized -> M17_GM300_RPi-rescue:C_Polarized-Device
- C3, C6, C7: footprint Capacitor_THT:CP_Radial_D8.0mm_P5.00mm -> Capacitor_SMD:C_0402_1005Metric
- C4, C5: footprint Capacitor_THT:C_Disc_D5.0mm_W2.5mm_P5.00mm -> Capacitor_SMD:C_0402_1005Metric
- D3: renamed from D2; footprint LED_THT:LED_D3.0mm -> LED_SMD:LED_0402_1005Metric
- D4: renamed from D3; footprint LED_THT:LED_D3.0mm -> LED_SMD:LED_0402_1005Metric
- D5: renamed from D4; footprint LED_THT:LED_D3.0mm -> LED_SMD:LED_0402_1005Metric
- J2: footprint CUI_SJ1-3523N -> parts:CUI_SJ1-3523N
- J3: footprint PHOENIX_1935161 -> parts:PHOENIX_1935161
- L1: renamed from L?; footprint (none) -> Inductor_SMD:L_0402_1005Metric
- Q1, Q2, Q3, Q4: footprint Package_TO_SOT_THT:TO-92_HandSolder -> Package_TO_SOT_SMD:SOT-23
- R1, R2, R3, R4, R5, R6, R7, R8, R9: footprint Resistor_THT:R_Axial_DIN0207_L6.3mm_D2.5mm_P7.62mm_Horizontal -> Resistor_SMD:R_0402_1005Metric
- U2: footprint (none) -> Package_SO:SOIC-16_3.9x9.9mm_P1.27mm
- U3: footprint (none) -> Package_SO:MSOP-8_3x3mm_P0.65mm
- gave numbers to parts that had none: 2
- renumbered D1 to D2

Commit message: initial pcb layout, change smds to 0603
Parts:
- C1, C2, C3, C4, C5, C6, C7: footprint Capacitor_SMD:C_0402_1005Metric -> Capacitor_SMD:C_0603_1608Metric
- D3, D4, D5: footprint LED_SMD:LED_0402_1005Metric -> LED_SMD:LED_0603_1608Metric
- L1: footprint Inductor_SMD:L_0402_1005Metric -> Inductor_SMD:L_0603_1608Metric
- R1, R2, R3, R4, R5, R6, R7, R8, R9: footprint Resistor_SMD:R_0402_1005Metric -> Resistor_SMD:R_0603_1608Metric
Changed lines of the file:
@@
 F 0 "D5" V 9189 1432 50  0000 R CNN
 F 1 "GRN" V 9098 1432 50  0000 R CNN
-F 2 "LED_SMD:LED_0402_1005Metric" H 9150 1550 50  0001 C CNN
+F 2 "LED_SMD:LED_0603_1608Metric" H 9150 1550 50  0001 C CNN
 F 3 "~" H 9150 1550 50  0001 C CNN
 	1    9150 1550
@@
 F 0 "D4" V 8839 1432 50  0000 R CNN
 F 1 "RED" V 8748 1432 50  0000 R CNN
-F 2 "LED_SMD:LED_0402_1005Metric" H 8800 1550 50  0001 C CNN
+F 2 "LED_SMD:LED_0603_1608Metric" H 8800 1550 50  0001 C CNN
 F 3 "~" H 8800 1550 50  0001 C CNN
 	1    8800 1550
@@
 F 0 "D3" V 8489 1432 50  0000 R CNN
 F 1 "BLU" V 8398 1432 50  0000 R CNN
-F 2 "LED_SMD:LED_0402_1005Metric" H 8450 1550 50  0001 C CNN
+F 2 "LED_SMD:LED_0603_1608Metric" H 8450 1550 50  0001 C CNN
 F 3 "~" H 8450 1550 50  0001 C CNN
 	1    8450 1550
@@
 F 0 "R8" H 9220 2046 50  0000 L CNN
 F 1 "2K2" H 9220 1955 50  0000 L CNN
-F 2 "Resistor_SMD:R_0402_1005Metric" V 9080 2000 50  0001 C CNN
+F 2 "Resistor_SMD:R_0603_1608Metric" V 9080 2000 50  0001 C CNN
 F 3 "~" H 9150 2000 50  0001 C CNN
 	1    9150 2000
@@
 F 0 "R7" H 8870 2046 50  0000 L CNN
 F 1 "1K" H 8870 1955 50  0000 L CNN
-F 2 "Resistor_SMD:R_0402_1005Metric" V 8730 2000 50  0001 C CNN
+F 2 "Resistor_SMD:R_0603_1608Metric" V 8730 2000 50  0001 C CNN
 F 3 "~" H 8800 2000 50  0001 C CNN
 	1    8800 2000
@@
 F 0 "R6" H 8520 2046 50  0000 L CNN
 F 1 "2K2" H 8520 1955 50  0000 L CNN
-F 2 "Resistor_SMD:R_0402_1005Metric" V 8380 2000 50  0001 C CNN
+F 2 "Resistor_SMD:R_0603_1608Metric" V 8380 2000 50  0001 C CNN
 F 3 "~" H 8450 2000 50  0001 C CNN
 	1    8450 2000
@@
 F 0 "R3" H 5920 1746 50  0000 L CNN
 F 1 "390R" H 5920 1655 50  0000 L CNN
-F 2 "Resistor_SMD:R_0402_1005Metric" V 5780 1700 50  0001 C CNN
+F 2 "Resistor_SMD:R_0603_1608Metric" V 5780 1700 50  0001 C CNN
 F 3 "~" H 5850 1700 50  0001 C CNN
 	1    5850 1700
@@
 F 0 "R4" V 5893 1300 50  0000 C CNN
 F 1 "680R" V 5984 1300 50  0000 C CNN
-F 2 "Resistor_SMD:R_0402_1005Metric" V 6030 1300 50  0001 C CNN
+F 2 "Resistor_SMD:R_0603_1608Metric" V 6030 1300 50  0001 C CNN
 F 3 "~" H 6100 1300 50  0001 C CNN
 	1    6100 1300
@@
 F 0 "C3" V 5345 1300 50  0000 C CNN
 F 1 "22u" V 5436 1300 50  0000 C CNN
-F 2 "Capacitor_SMD:C_0402_1005Metric" H 5638 1150 50  0001 C CNN
+F 2 "Capacitor_SMD:C_0603_1608Metric" H 5638 1150 50  0001 C CNN
 F 3 "~" H 5600 1300 50  0001 C CNN
 	1    5600 1300
@@
 F 0 "C4" H 8515 4146 50  0000 L CNN
 F 1 "220n" H 8515 4055 50  0000 L CNN
-F 2 "Capacitor_SMD:C_0402_1005Metric" H 8438 3950 50  0001 C CNN
+F 2 "Capacitor_SMD:C_0603_1608Metric" H 8438 3950 50  0001 C CNN
 F 3 "~" H 8400 4100 50  0001 C CNN
 	1    8400 4100
@@
 F 0 "C7" H 10368 4146 50  0000 L CNN
 F 1 "47u" H 10368 4055 50  0000 L CNN
-F 2 "Capacitor_SMD:C_0402_1005Metric" H 10288 3950 50  0001 C CNN
+F 2 "Capacitor_SMD:C_0603_1608Metric" H 10288 3950 50  0001 C CNN
 F 3 "~" H 10250 4100 50  0001 C CNN
 	1    10250 4100
@@
 F 0 "R9" H 10620 5696 50  0000 L CNN
 F 1 "22K" H 10620 5605 50  0000 L CNN
-F 2 "Resistor_SMD:R_0402_1005Metric" V 10480 5650 50  0001 C CNN
+F 2 "Resistor_SMD:R_0603_1608Metric" V 10480 5650 50  0001 C CNN
 F 3 "~" H 10550 5650 50  0001 C CNN
 	1    10550 5650
@@
 F 0 "C6" V 9755 5900 50  0000 C CNN
 F 1 "220u" V 9664 5900 50  0000 C CNN
-F 2 "Capacitor_SMD:C_0402_1005Metric" H 9538 5750 50  0001 C CNN
+F 2 "Capacitor_SMD:C_0603_1608Metric" H 9538 5750 50  0001 C CNN
 F 3 "~" H 9500 5900 50  0001 C CNN
 	1    9500 5900
@@
 F 0 "C5" V 8248 5800 50  0000 C CNN
 F 1 "470n" V 8339 5800 50  0000 C CNN
-F 2 "Capacitor_SMD:C_0402_1005Metric" H 8538 5650 50  0001 C CNN
+F 2 "Capacitor_SMD:C_0603_1608Metric" H 8538 5650 50  0001 C CNN
 F 3 "~" H 8500 5800 50  0001 C CNN
 	1    8500 5800
@@
 F 0 "R5" V 7743 5550 50  0000 C CNN
 F 1 "39K" V 7834 5550 50  0000 C CNN
-F 2 "Resistor_SMD:R_0402_1005Metric" V 7880 5550 50  0001 C CNN
+F 2 "Resistor_SMD:R_0603_1608Metric" V 7880 5550 50  0001 C CNN
 F 3 "~" H 7950 5550 50  0001 C CNN
 	1    7950 5550
@@
 F 0 "R1" H 4570 5846 50  0000 L CNN
 F 1 "47K" H 4570 5755 50  0000 L CNN
-F 2 "Resistor_SMD:R_0402_1005Metric" V 4430 5800 50  0001 C CNN
+F 2 "Resistor_SMD:R_0603_1608Metric" V 4430 5800 50  0001 C CNN
 F 3 "~" H 4500 5800 50  0001 C CNN
 	1    4500 5800
@@
 F 0 "R2" H 5320 5846 50  0000 L CNN
 F 1 "47K" H 5320 5755 50  0000 L CNN
-F 2 "Resistor_SMD:R_0402_1005Metric" V 5180 5800 50  0001 C CNN
+F 2 "Resistor_SMD:R_0603_1608Metric" V 5180 5800 50  0001 C CNN
 F 3 "~" H 5250 5800 50  0001 C CNN
 	1    5250 5800
@@
 F 0 "C1" H 1718 1646 50  0000 L CNN
 F 1 "100 uF" H 1718 1555 50  0000 L CNN
-F 2 "Capacitor_SMD:C_0402_1005Metric" H 1638 1450 50  0001 C CNN
+F 2 "Capacitor_SMD:C_0603_1608Metric" H 1638 1450 50  0001 C CNN
 F 3 "~" H 1600 1600 50  0001 C CNN
 	1    1600 1600
@@
 F 0 "L1" V 3490 1500 50  0000 C CNN
 F 1 "100 uH" V 3399 1500 50  0000 C CNN
-F 2 "Inductor_SMD:L_0402_1005Metric" H 3300 1500 50  0001 C CNN
+F 2 "Inductor_SMD:L_0603_1608Metric" H 3300 1500 50  0001 C CNN
 F 3 "~" H 3300 1500 50  0001 C CNN
 	1    3300 1500
@@
 F 0 "C2" H 3568 1696 50  0000 L CNN
 F 1 "1000 uF" H 3568 1605 50  0000 L CNN
-F 2 "Capacitor_SMD:C_0402_1005Metric" H 3488 1500 50  0001 C CNN
+F 2 "Capacitor_SMD:C_0603_1608Metric" H 3488 1500 50  0001 C CNN
 F 3 "~" H 3450 1650 50  0001 C CNN
 	1    3450 1650
